File: Hardware Design Files/Speaker/Speaker.kicad_sch (KiCad schematic)
At the start: 23 parts, among them J1 Conn_01x08_Pin, J2 Conn_01x08_Pin, J3 Screw_Terminal_01x07, U1 LMV358IDR, U2 MAX5187BEEG+, U3 PAM8304, U4 PAM8304, U5 PAM8304

Commit message: changed R1
changed from 10k to 70k such that chip select current ~5ua
Parts:
- R1: value 10K -> 70K; DIGIKEY PART # RMCF0805FT10K0 -> ERJ-1GNF6982C
Changed lines of the file:
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@@
       (effects (font (size 1.27 1.27)) (justify right))
     )
-    (property "Value" "10K" (at 31.115 76.2 0)
+    (property "Value" "70K" (at 31.115 76.2 0)
       (effects (font (size 1.27 1.27)) (justify right))
     )
@@
       (effects (font (size 1.27 1.27)) hide)
     )
-    (property "Datasheet" "~https://www.seielect.com/catalog/sei-rmcf_rmcp.pdf" (at 28.575 74.93 0)
+    (property "Datasheet" "https://industrial.panasonic.com/cdbs/www-data/pdf/RDA0000/AOA0000C304.pdf" (at 28.575 74.93 0)
       (effects (font (size 1.27 1.27)) hide)
     )
-    (property "DIGIKEY PART #" "RMCF0805FT10K0" (at 28.575 74.93 0)
+    (property "DIGIKEY PART #" "ERJ-1GNF6982C" (at 28.575 74.93 0)
       (effects (font (size 1.27 1.27)) hide)
     )
