File: Hardware Design Files/power_electronics/buck_converter_3v/_autosave-buck_converter_3v.kicad_sch (KiCad schematic)
At the start: 22 parts, among them J1 Conn_01x02, J2 Conn_01x02

Commit message: feat(buck_converter_3v): select specific parts on digikey
Parts:
- J1, J2: footprint (none) -> custom_footprints:2-terminal-screw-connector-691137710002; Digikey PN (none) -> 691137710002
Changed lines of the file:
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@@
       (effects (font (size 1.27 1.27)) (justify left))
     )
-    (property "Footprint" "" (at 249.555 32.385 0)
+    (property "Footprint" "custom_footprints:2-terminal-screw-connector-691137710002" (at 249.555 32.385 0)
       (effects (font (size 1.27 1.27)) hide)
     )
@@
       (effects (font (size 1.27 1.27)) hide)
     )
-    (property "Digikey PN" "" (at 249.555 32.385 0)
+    (property "Digikey PN" "691137710002" (at 249.555 32.385 0)
       (effects (font (size 1.27 1.27)) hide)
     )
@@
       (effects (font (size 1.27 1.27)))
     )
-    (property "Footprint" "" (at 19.05 34.925 0)
+    (property "Footprint" "custom_footprints:2-terminal-screw-connector-691137710002" (at 19.05 34.925 0)
       (effects (font (size 1.27 1.27)) hide)
     )
@@
       (effects (font (size 1.27 1.27)) hide)
     )
-    (property "Digikey PN" "" (at 19.05 34.925 0)
-      (effects (font (size 1.27 1.27)) hide)
-    )
+    (property "Digikey PN" "691137710002" (at 19.05 34.925 0)
+      (effects (font (size 1.27 1.27)) hide)
+    )
