File: Hardware Design Files/power_electronics/buck_converter_3v/buck_converter_3v.kicad_sch (KiCad schematic)
At the start: 22 parts, among them J1 Conn_01x02, J2 Conn_01x02

Commit message: feat(buck_converter_3v): create PCB
Parts:
- J1, J2: footprint (none) -> custom_footprints:2-terminal-screw-connector-691137710002; Digikey PN (none) -> 691137710002
- PS1: footprint LM61495QRPHRQ1:CONV_LM61495QRPHRQ1 -> custom_footprints:CONV_LM61495QRPHRQ1
- renumbered Cboot to Cboot1, Cff to Cff1, Cvcc to Cvcc1, Rfbb to Rfbb1, Rfbt to Rfbt1, Rff to Rff1, Rreset to Rreset1
Connections:
- net Vout: now reaches Cout1.1, Cout2.1, Cout3.1, Cout4.1, Cout5.1, Cout6.1, Cout7.1, J2.1 (Pin_1), L1.2, PS1.5 (BIAS), Rfbt1.1, Rff1.1, Rreset1.1
- net Vin: now reaches Cin1.1, Cin2.1, Cin_hf1.1, Cin_hf2.1, J1.2 (Pin_2), PS1.13 (EN), PS1.14 (VIN1), PS1.2 (VIN2)
- net switch_out: now reaches Cboot1.1, L1.1, PS1.16 (SW)

Commit message: feat(buck_converter): unify pcb design, schematic varies by resistor value, add mounting holes
Parts:
- removed Rfbb1: 46.5k, Resistor_SMD:R_0805_2012Metric, symbol Device:R
- added H1, H2, H3, H4: MountingHole, MountingHole:MountingHole_2.5mm_Pad, symbol Mechanical:MountingHole
- added Rfbb2: 46.5k, Resistor_SMD:R_0805_2012Metric, symbol Device:R
- L1: value 2.2u -> 3.3u
Connections:
- net GND: now also Rfbb2.2
- net at Cff1.2, PS1.7 (FB), Rfbt1.2: now also Rfbb2.1
Changed lines of the file:
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@@
+    )
+  )
+  (symbol (lib_id "Mechanical:MountingHole") (at 22.225 90.805 0) (unit 1)
+    (in_bom yes) (on_board yes) (dnp no) (fields_autoplaced)
+    (property "Reference" "H1" (at 25.4 89.535 0)
+      (effects (font (size 1.27 1.27)) (justify left))
+    )
+    (property "Value" "MountingHole" (at 25.4 92.075 0)
+      (effects (font (size 1.27 1.27)) (justify left))
+    )
+    (property "Footprint" "MountingHole:MountingHole_2.5mm_Pad" (at 22.225 90.805 0)
+      (effects (font (size 1.27 1.27)) hide)
+    )
+    (property "Datasheet" "~" (at 22.225 90.805 0)
+      (effects (font (size 1.27 1.27)) hide)
+    )
+    (instances
+      (project "buck_converter_3v"
+        (path "/666415fd-4643-4739-b592-9d5f83af5eff"
+          (reference "H1") (unit 1)
+        )
+      )
     )
   )
@@
     )
   )
+  (symbol (lib_id "Mechanical:MountingHole") (at 22.225 107.315 0) (unit 1)
+    (in_bom yes) (on_board yes) (dnp no) (fields_autoplaced)
+    (property "Reference" "H4" (at 25.4 106.045 0)
+      (effects (font (size 1.27 1.27)) (justify left))
+    )
+    (property "Value" "MountingHole" (at 25.4 108.585 0)
+      (effects (font (size 1.27 1.27)) (justify left))
+    )
+    (property "Footprint" "MountingHole:MountingHole_2.5mm_Pad" (at 22.225 107.315 0)
+      (effects (font (size 1.27 1.27)) hide)
+    )
+    (property "Datasheet" "~" (at 22.225 107.315 0)
+      (effects (font (size 1.27 1.27)) hide)
+    )
+    (instances
+      (project "buck_converter_3v"
+        (path "/666415fd-4643-4739-b592-9d5f83af5eff"
+          (reference "H4") (unit 1)
+        )
+      )
+    )
+  )
   (symbol (lib_id "power:GND") (at 227.965 81.915 0) (unit 1)
     (in_bom yes) (on_board yes) (dnp no) (fields_autoplaced)
@@
     )
   )
-  (symbol (lib_id "Device:R") (at 227.965 78.105 0) (unit 1)
-    (in_bom yes) (on_board yes) (dnp no) (fields_autoplaced)
-    (property "Reference" "Rfbb1" (at 230.505 76.835 0)
-      (effects (font (size 1.27 1.27)) (justify left))
-    )
-    (property "Value" "46.5k" (at 230.505 79.375 0)
-      (effects (font (size 1.27 1.27)) (justify left))
-    )
-    (property "Footprint" "Resistor_SMD:R_0805_2012Metric" (at 226.187 78.105 90)
-      (effects (font (size 1.27 1.27)) hide)
-    )
-    (property "Datasheet" "~" (at 227.965 78.105 0)
-      (effects (font (size 1.27 1.27)) hide)
-    )
-    (property "Digikey PN" "ERA-6AEB4642V" (at 227.965 78.105 0)
-      (effects (font (size 1.27 1.27)) hide)
-    )
-    (pin "2")
-    (pin "1")
-    (instances
-      (project "buck_converter_3v"
-        (path "/666415fd-4643-4739-b592-9d5f83af5eff"
-          (reference "Rfbb1") (unit 1)
-        )
-      )
-    )
-  )
   (symbol (lib_id "Device:C") (at 135.89 56.515 0) (unit 1)
     (in_bom yes) (on_board yes) (dnp no) (fields_autoplaced)
@@
     )
   )
+  (symbol (lib_id "Mechanical:MountingHole") (at 22.225 96.52 0) (unit 1)
+    (in_bom yes) (on_board yes) (dnp no) (fields_autoplaced)
+    (property "Reference" "H2" (at 25.4 95.25 0)
+      (effects (font (size 1.27 1.27)) (justify left))
+    )
+    (property "Value" "MountingHole" (at 25.4 97.79 0)
+      (effects (font (size 1.27 1.27)) (justify left))
+    )
+    (property "Footprint" "MountingHole:MountingHole_2.5mm_Pad" (at 22.225 96.52 0)
+      (effects (font (size 1.27 1.27)) hide)
+    )
+    (property "Datasheet" "~" (at 22.225 96.52 0)
+      (effects (font (size 1.27 1.27)) hide)
+    )
+    (instances
+      (project "buck_converter_3v"
+        (path "/666415fd-4643-4739-b592-9d5f83af5eff"
+          (reference "H2") (unit 1)
+        )
+      )
+    )
+  )
   (symbol (lib_id "Device:L") (at 128.905 52.705 90) (unit 1)
     (in_bom yes) (on_board yes) (dnp no) (fields_autoplaced)
-    (property "Reference" "L1" (at 128.905 47.625 90)
-      (effects (font (size 1.27 1.27)))
-    )
-    (property "Value" "2.2u" (at 128.905 50.165 90)
+    (property "Reference" "L1" (at 128.905 46.99 90)
+      (effects (font (size 1.27 1.27)))
+    )
+    (property "Value" "3.3u" (at 128.905 49.53 90)
       (effects (font (size 1.27 1.27)))
     )
@@
     )
   )
+  (symbol (lib_id "Mechanical:MountingHole") (at 22.225 102.235 0) (unit 1)
+    (in_bom yes) (on_board yes) (dnp no) (fields_autoplaced)
+    (property "Reference" "H3" (at 25.4 100.965 0)
+      (effects (font (size 1.27 1.27)) (justify left))
+    )
+    (property "Value" "MountingHole" (at 25.4 103.505 0)
+      (effects (font (size 1.27 1.27)) (justify left))
+    )
+    (property "Footprint" "MountingHole:MountingHole_2.5mm_Pad" (at 22.225 102.235 0)
+      (effects (font (size 1.27 1.27)) hide)
+    )
+    (property "Datasheet" "~" (at 22.225 102.235 0)
+      (effects (font (size 1.27 1.27)) hide)
+    )
+    (instances
+      (project "buck_converter_3v"
+        (path "/666415fd-4643-4739-b592-9d5f83af5eff"
+          (reference "H3") (unit 1)
+        )
+      )
+    )
+  )
   (symbol (lib_id "power:GND") (at 64.77 80.645 0) (unit 1)
     (in_bom yes) (on_board yes) (dnp no) (fields_autoplaced)
@@
         )
       )
+    )
+  )
+  (symbol (lib_id "Device:R") (at 227.965 78.105 0) (unit 1)
+    (in_bom yes) (on_board yes) (dnp no) (fields_autoplaced)
+    (property "Reference" "Rfbb2" (at 230.505 76.835 0)
+      (effects (font (size 1.27 1.27)) (justify left))
+    )
+    (property "Value" "46.5k" (at 230.505 79.375 0)
+      (effects (font (size 1.27 1.27)) (justify left))
+    )
+    (property "Footprint" "Resistor_SMD:R_0805_2012Metric" (at 226.187 78.105 90)
+      (effects (font (size 1.27 1.27)) hide)
+    )
+    (property "Datasheet" "~" (at 227.965 78.105 0)
+      (effects (font (size 1.27 1.27)) hide)
+    )
+    (property "Digikey PN" "ERA-6AEB4642V" (at 227.965 78.105 0)
+      (effects (font (size 1.27 1.27)) hide)
+    )
+    (pin "2")
+    (pin "1")
+    (instances
+      (project "buck_converter_3v"
+        (path "/666415fd-4643-4739-b592-9d5f83af5eff"
+          (reference "Rfbb2") (unit 1)
+        )
+      )
